Commit message: feat: add DG5F-S bimanual RL asset; fix link7 motor mesh and mount plane
- vendor/tesollo_model: import latest DG5F-S vendor URDFs + meshes
- tools/gen_dg5fs_xacro.py: side-prefixed DG5F-S fragments with the DG5F
  adapter plate inserted (chain mirrors DG5F incl. palm slots)
- openarm_tesollo_bi_s(+_rl): new DG5F-S bimanual asset, 54D action,
  manifest joint/link parity with the DG5F asset
- generate_rl_urdf.py: swap stock link7 meshes for cropped variants on any
  link7 carrying a hand mount (stock-gripper motor section removed)
- tesollo mounts seated on the link7 flange plate plane (z=0.0495); the
  flange bolts insert into the adapter plate holes

File: assemblies/openarm_modular_dual_tesollo.xacro (robot description, xacro)
@@ -19,7 +19,7 @@
   <xacro:arg name="ee_type" default="none"/>
   <!-- Mount transforms -->
-  <xacro:arg name="left_mount_xyz" default="0 0 0.0595695"/>
+  <xacro:arg name="left_mount_xyz" default="0 0 0.0495"/>
   <xacro:arg name="left_mount_rpy" default="0 0 1.5707964"/>
-  <xacro:arg name="right_mount_xyz" default="0 0.0000003 0.0595695"/>
+  <xacro:arg name="right_mount_xyz" default="0 0.0000003 0.0495"/>
   <xacro:arg name="right_mount_rpy" default="0 0 -1.5707964"/>
   <!-- Optional: upstream Tesollo xacro paths -->

File: generated/rl/openarm_tesollo_bi_rl.urdf (robot description, URDF)
Before this commit: robot openarm_dual_tesollo_rl, 84 links, 83 joints
Joints:
- joint l_hj_mount: origin xyz=0 0 0.0595695 rpy=0 0 1.5707964 -> xyz=0 0 0.0495 rpy=0 0 1.5707964
- joint r_hj_mount: origin xyz=0 0.0000003 0.0595695 rpy=0 0 -1.5707964 -> xyz=0 0.0000003 0.0495 rpy=0 0 -1.5707964

File: generated/rl/openarm_tesollo_sensor_rl.urdf (robot description, URDF)
Before this commit: robot openarm_tesollo_sensor_rl, 57 links, 56 joints
Joints:
- joint r_hj_mount: origin xyz=0 0.0000003 0.0595695 rpy=0 0 -1.5707964 -> xyz=0 0.0000003 0.0495 rpy=0 0 -1.5707964

File: generated/source/openarm_tesollo_bi.urdf (robot description, URDF)
Before this commit: robot openarm_dual_tesollo, 80 links, 79 joints
Joints:
- joint mount_left_link7_to_tesollo: origin xyz=0 0 0.0595695 rpy=0 0 1.5707964 -> xyz=0 0 0.0495 rpy=0 0 1.5707964
- joint mount_right_link7_to_tesollo: origin xyz=0 0.0000003 0.0595695 rpy=0 0 -1.5707964 -> xyz=0 0.0000003 0.0495 rpy=0 0 -1.5707964

File: generated/source/openarm_tesollo_sensor.urdf (robot description, URDF)
Before this commit: robot openarm_tesollo_sensor, 53 links, 52 joints
Joints:
- joint mount_right_link7_to_tesollo: origin xyz=0 0.0000003 0.0595695 rpy=0 0 -1.5707964 -> xyz=0 0.0000003 0.0495 rpy=0 0 -1.5707964
