Commit message: feat: self-collision-safe asset pipeline - audit, headless USD build, fabric URDFs
- tools/audit_self_collision.py: permanent resting-penetration audit
  (PhysX non-adjacent pairing, raw FAIL / hull-only WARN, allowlist with
  accept_raw); runs inside generate_rl_urdf.py
- tools/build_usd.py: headless UrdfConverter build (convex_decomposition,
  merge_fixed_joints, fix_base pinned), manifest joint/collider contract
  check, PhysicsFilteredPairsAPI authored from manifest
  self_collision_filtered_pairs (cooking inflation ate a 2.8mm clearance ->
  4kN phantom contacts), per-asset self-contained bundles, --sync-hdgp
- tools/gen_fabric_urdfs.py: consolidates the four hdgp fabric generators;
  kinematics patched from RL URDFs (legacy +8mm arm base fixed), FK-gated
- RH56F1: unrepairable non-watertight collisions replaced with fitted
  primitives (inscribed cylinders/boxes, palm_1 cover dropped)
- tools/probe_zero_action.py: zero-action drift probe - all four assets hold
  <1e-5 rad over 200 steps with enabled_self_collisions=True

File: generated/rl/openarm_bi_rh56f1_rl.urdf (robot description, URDF)
Before this commit: robot openarm_bi_rh56f1_rl, 76 links, 75 joints
Links:
- link l_al_7: geometry collision mesh filename=file:///home/user/rl_ws/urdf/generated/rl/meshes/link7_flan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 scale=0.001 -0.001 0.001; visual mesh filename=file:///home/user/rl_ws/urdf/vendor/openarm_description/mes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 scale=0.001 -0.001 0.001
- link l_hl_index_1: geometry collision cylinder length=0.0463133 radius=0.00806266; visual mesh filename=file:///home/user/rl_ws/urdf/vendor/RH56F1/RH56F1_L/meshes/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
- link l_hl_index_2: geometry collision cylinder length=0.0502971 radius=0.00723799; visual mesh filename=file:///home/user/rl_ws/urdf/vendor/RH56F1/RH56F1_L/meshes/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
- link l_hl_index_sensor: geometry collision cylinder length=0.0507537 radius=0.00817662; visual mesh filename=file:///home/user/rl_ws/urdf/vendor/RH56F1/RH56F1_L/meshes/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
- link l_hl_index_tip: geometry collision box size=0.0160206 0.0456063 0.0292686; visual mesh filename=file:///home/user/rl_ws/urdf/vendor/RH56F1/RH56F1_L/meshes/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
- link l_hl_middle_1: geometry collision cylinder length=0.0463133 radius=0.00806266; visual mesh filename=file:///home/user/rl_ws/urdf/vendor/RH56F1/RH56F1_L/meshes/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
- link l_hl_middle_2: geometry collision cylinder length=0.0532292 radius=0.00723601; visual mesh filename=file:///home/user/rl_ws/urdf/vendor/RH56F1/RH56F1_L/meshes/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
- link l_hl_middle_sensor: geometry collision cylinder length=0.0536642 radius=0.00729131; visual mesh filename=file:///home/user/rl_ws/urdf/vendor/RH56F1/RH56F1_L/meshes/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
- link l_hl_middle_tip: geometry collision box size=0.014472 0.0483447 0.0305089; visual mesh filename=file:///home/user/rl_ws/urdf/vendor/RH56F1/RH56F1_L/meshes/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
- link l_hl_palm_1: geometry visual mesh filename=file:///home/user/rl_ws/urdf/vendor/RH56F1/RH56F1_L/meshes/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
- link l_hl_pinky_1: geometry collision cylinder length=0.0463133 radius=0.00806266; visual mesh filename=file:///home/user/rl_ws/urdf/vendor/RH56F1/RH56F1_L/meshes/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
- link l_hl_pinky_2: geometry collision cylinder length=0.0432787 radius=0.00716796; visual mesh filename=file:///home/user/rl_ws/urdf/vendor/RH56F1/RH56F1_L/meshes/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
- link l_hl_pinky_sensor: geometry collision cylinder length=0.0438574 radius=0.00795973; visual mesh filename=file:///home/user/rl_ws/urdf/vendor/RH56F1/RH56F1_L/meshes/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
- link l_hl_pinky_tip: geometry collision box size=0.0161707 0.0393926 0.0264591; visual mesh filename=file:///home/user/rl_ws/urdf/vendor/RH56F1/RH56F1_L/meshes/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
- link l_hl_ring_1: geometry collision cylinder length=0.0463133 radius=0.00806266; visual mesh filename=file:///home/user/rl_ws/urdf/vendor/RH56F1/RH56F1_L/meshes/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
- link l_hl_ring_2: geometry collision cylinder length=0.0502971 radius=0.00723799; visual mesh filename=file:///home/user/rl_ws/urdf/vendor/RH56F1/RH56F1_L/meshes/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
- link l_hl_ring_sensor: geometry collision cylinder length=0.0507024 radius=0.00770788; visual mesh filename=file:///home/user/rl_ws/urdf/vendor/RH56F1/RH56F1_L/meshes/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
- link l_hl_ring_tip: geometry collision box size=0.015568 0.0456113 0.0293262; visual mesh filename=file:///home/user/rl_ws/urdf/vendor/RH56F1/RH56F1_L/meshes/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
- link l_hl_thumb_1: geometry collision box size=0.00761364 0.0206182 0.0153284; visual mesh filename=file:///home/user/rl_ws/urdf/vendor/RH56F1/RH56F1_L/meshes/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
- link l_hl_thumb_2: geometry collision box size=0.0583821 0.0598939 0.0222501; visual mesh filename=file:///home/user/rl_ws/urdf/vendor/RH56F1/RH56F1_L/meshes/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
- link l_hl_thumb_3: geometry collision box size=0.0340982 0.0371097 0.0202092; visual mesh filename=file:///home/user/rl_ws/urdf/vendor/RH56F1/RH56F1_L/meshes/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
- link l_hl_thumb_4: geometry collision box size=0.0243792 0.0336509 0.0162755; visual mesh filename=file:///home/user/rl_ws/urdf/vendor/RH56F1/RH56F1_L/meshes/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
- link l_hl_thumb_sensor: geometry collision cylinder length=0.0364273 radius=0.00856693; visual mesh filename=file:///home/user/rl_ws/urdf/vendor/RH56F1/RH56F1_L/meshes/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
- link l_hl_thumb_tip: geometry collision box size=0.0162751 0.0297926 0.0297745; visual mesh filename=file:///home/user/rl_ws/urdf/vendor/RH56F1/RH56F1_L/meshes/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
- link r_al_7: geometry collision mesh filename=file:///home/user/rl_ws/urdf/generated/rl/meshes/link7_flan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 scale=0.001 0.001 0.001; visual mesh filename=file:///home/user/rl_ws/urdf/vendor/openarm_description/mes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 scale=0.001 0.001 0.001
- link r_hl_index_1: geometry collision cylinder length=0.0463133 radius=0.00806266; visual mesh filename=file:///home/user/rl_ws/urdf/vendor/RH56F1/RH56F1_R/meshes/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
- link r_hl_index_2: geometry collision cylinder length=0.0502971 radius=0.0072377; visual mesh filename=file:///home/user/rl_ws/urdf/vendor/RH56F1/RH56F1_R/meshes/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
- link r_hl_index_sensor: geometry collision cylinder length=0.0507241 radius=0.0079409; visual mesh filename=file:///home/user/rl_ws/urdf/vendor/RH56F1/RH56F1_R/meshes/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
- link r_hl_index_tip: geometry collision box size=0.0157954 0.0456248 0.0293267; visual mesh filename=file:///home/user/rl_ws/urdf/vendor/RH56F1/RH56F1_R/meshes/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
- link r_hl_middle_1: geometry collision cylinder length=0.0463133 radius=0.00806266; visual mesh filename=file:///home/user/rl_ws/urdf/vendor/RH56F1/RH56F1_R/meshes/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
- link r_hl_middle_2: geometry collision cylinder length=0.0532292 radius=0.00723557; visual mesh filename=file:///home/user/rl_ws/urdf/vendor/RH56F1/RH56F1_R/meshes/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
- link r_hl_middle_sensor: geometry collision cylinder length=0.0536642 radius=0.0072913; visual mesh filename=file:///home/user/rl_ws/urdf/vendor/RH56F1/RH56F1_R/meshes/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
- link r_hl_middle_tip: geometry collision box size=0.0144707 0.0483447 0.0305088; visual mesh filename=file:///home/user/rl_ws/urdf/vendor/RH56F1/RH56F1_R/meshes/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
- link r_hl_palm_1: geometry visual mesh filename=file:///home/user/rl_ws/urdf/vendor/RH56F1/RH56F1_R/meshes/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
- link r_hl_pinky_1: geometry collision cylinder length=0.0463133 radius=0.00806266; visual mesh filename=file:///home/user/rl_ws/urdf/vendor/RH56F1/RH56F1_R/meshes/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
- link r_hl_pinky_2: geometry collision cylinder length=0.0432787 radius=0.00716796; visual mesh filename=file:///home/user/rl_ws/urdf/vendor/RH56F1/RH56F1_R/meshes/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
- link r_hl_pinky_sensor: geometry collision cylinder length=0.043889 radius=0.00797037; visual mesh filename=file:///home/user/rl_ws/urdf/vendor/RH56F1/RH56F1_R/meshes/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
- link r_hl_pinky_tip: geometry collision box size=0.0161457 0.0394019 0.026465; visual mesh filename=file:///home/user/rl_ws/urdf/vendor/RH56F1/RH56F1_R/meshes/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
- link r_hl_ring_1: geometry collision cylinder length=0.0463133 radius=0.00806266; visual mesh filename=file:///home/user/rl_ws/urdf/vendor/RH56F1/RH56F1_R/meshes/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
- link r_hl_ring_2: geometry collision cylinder length=0.0502971 radius=0.0072377; visual mesh filename=file:///home/user/rl_ws/urdf/vendor/RH56F1/RH56F1_R/meshes/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
- link r_hl_ring_sensor: geometry collision cylinder length=0.0507444 radius=0.00803594; visual mesh filename=file:///home/user/rl_ws/urdf/vendor/RH56F1/RH56F1_R/meshes/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
- link r_hl_ring_tip: geometry collision box size=0.0155468 0.045617 0.0293267; visual mesh filename=file:///home/user/rl_ws/urdf/vendor/RH56F1/RH56F1_R/meshes/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
- link r_hl_thumb_1: geometry collision box size=0.00758285 0.0205866 0.0153284; visual mesh filename=file:///home/user/rl_ws/urdf/vendor/RH56F1/RH56F1_R/meshes/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
- link r_hl_thumb_2: geometry collision box size=0.0544741 0.0620779 0.0222501; visual mesh filename=file:///home/user/rl_ws/urdf/vendor/RH56F1/RH56F1_R/meshes/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
- link r_hl_thumb_3: geometry collision box size=0.0340982 0.0371117 0.0202091; visual mesh filename=file:///home/user/rl_ws/urdf/vendor/RH56F1/RH56F1_R/meshes/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
- link r_hl_thumb_4: geometry collision box size=0.0243792 0.0336562 0.0162755; visual mesh filename=file:///home/user/rl_ws/urdf/vendor/RH56F1/RH56F1_R/meshes/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
- link r_hl_thumb_sensor: geometry collision cylinder length=0.0364273 radius=0.00856687; visual mesh filename=file:///home/user/rl_ws/urdf/vendor/RH56F1/RH56F1_R/meshes/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
- link r_hl_thumb_tip: geometry collision box size=0.0162752 0.0297899 0.0297747; visual mesh filename=file:///home/user/rl_ws/urdf/vendor/RH56F1/RH56F1_R/meshes/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

File: generated/rl/openarm_tesollo_bi_rl.urdf (robot description, URDF)
Before this commit: robot openarm_dual_tesollo_rl, 84 links, 83 joints
Links:
- link l_al_7: geometry collision mesh filename=file:///home/user/rl_ws/urdf/generated/rl/meshes/link7_flan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 scale=0.001 -0.001 0.001; visual mesh filename=file:///home/user/rl_ws/urdf/vendor/openarm_description/mes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 scale=0.001 -0.001 0.001
- link l_hl_adapter: geometry visual mesh filename=file:///home/user/rl_ws/urdf/install/dg_description/share/d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
- link r_al_7: geometry collision mesh filename=file:///home/user/rl_ws/urdf/generated/rl/meshes/link7_flan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 scale=0.001 0.001 0.001; visual mesh filename=file:///home/user/rl_ws/urdf/vendor/openarm_description/mes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 scale=0.001 0.001 0.001
- link r_hl_adapter: geometry visual mesh filename=file:///home/user/rl_ws/urdf/install/dg_description/share/d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

File: generated/rl/openarm_tesollo_bi_s_rl.urdf (robot description, URDF)
Before this commit: robot openarm_dual_tesollo_s_rl, 84 links, 83 joints
Links:
- link l_al_7: geometry collision mesh filename=file:///home/user/rl_ws/urdf/generated/rl/meshes/link7_flan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 scale=0.001 -0.001 0.001; visual mesh filename=file:///home/user/rl_ws/urdf/vendor/openarm_description/mes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 scale=0.001 -0.001 0.001
- link l_hl_adapter: geometry visual mesh filename=file:///home/user/rl_ws/urdf/vendor/delto_m_ros2/dg_descrip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
- link r_al_7: geometry collision mesh filename=file:///home/user/rl_ws/urdf/generated/rl/meshes/link7_flan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 scale=0.001 0.001 0.001; visual mesh filename=file:///home/user/rl_ws/urdf/vendor/openarm_description/mes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 scale=0.001 0.001 0.001
- link r_hl_adapter: geometry visual mesh filename=file:///home/user/rl_ws/urdf/vendor/delto_m_ros2/dg_descrip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

File: generated/rl/openarm_tesollo_sensor_rl.urdf (robot description, URDF)
Before this commit: robot openarm_tesollo_sensor_rl, 57 links, 56 joints
Links:
- link r_al_7: geometry collision mesh filename=file:///home/user/rl_ws/urdf/generated/rl/meshes/link7_flan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 scale=0.001 0.001 0.001; visual mesh filename=file:///home/user/rl_ws/urdf/vendor/openarm_description/mes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 scale=0.001 0.001 0.001
- link r_hl_adapter: geometry visual mesh filename=file:///home/user/rl_ws/urdf/install/dg_description/share/d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
